File: benchbuddy.kicad_pcb (KiCad board)
At the start: 2 copper layers, 0 parts

Commit message: Draw board outline in layout
Other:
- board outline added: 68.6 x 53.3 mm
Changed lines of the file:
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@@
     (area 0 0 0 0)
     (thickness 1.6)
-    (drawings 0)
+    (drawings 4)
     (tracks 0)
     (zones 0)
@@
     (add_net "")
   )
+  (gr_line (start 127 175.26) (end 127 121.92) (angle 90) (layer Edge.Cuts) (width 0.1))
+  (gr_line (start 195.58 175.26) (end 127 175.26) (angle 90) (layer Edge.Cuts) (width 0.1))
+  (gr_line (start 195.58 121.92) (end 195.58 175.26) (angle 90) (layer Edge.Cuts) (width 0.1))
+  (gr_line (start 127 121.92) (end 195.58 121.92) (angle 90) (layer Edge.Cuts) (width 0.1))
 )
